File: body_pads/out/forearm/forearm_Back.kicad_pcb (KiCad board)
At the start: 2 copper layers, 197.6 x 230.1 mm, 0 parts

Commit message: Terminate body pads with vias and an FFC connector; export the full Gerber set
The pad tails now follow README Step 5 like the glove: every electrode trace
ends in a through via (0.45/0.2 mm, two staggered rows) and a 16-pin 0.5 mm
FFC connector (KiCad library Hirose FH12-16S-0.5SH) sits on the side opposite
the electrodes, making each board a 2-layer flex. A nested staircase fans the
0.5 mm bus out to the 1.0 mm via pitch and back to the 0.5 mm pads without
crossings. body_pads/kicad_post.py runs with KiCad's own python to add the
vias, footprint, connector-side tracks and nets; a .kicad_pro with flex rules
is written so kicad-cli DRC checks the right limits, and the Gerber export now
produces the same file set as the glove (both copper layers, mask, paste,
silkscreen, edge cuts, Eco1/Eco2, PTH/NPTH drills and maps).

Also: the column grid is shifted so no column exits under the tail bus, the
mirrored chest half swaps its tail order so both halves match, previews gain
a tail close-up, and the README describes the new tail, layers and checks.
Includes the body-pad documentation docx added to the working tree.

Co-Authored-By: Claude Fable 5.1 <noreply@anthropic.com>
Parts:
- added J1: Hirose_FH12-16S-0.5SH_1x16-1MP_P0.50mm_Horizontal, Hirose_FH12-16S-0.5SH_1x16-1MP_P0.50mm_Horizontal, F.Cu at (119.3, 15.5)
Routing:
- net ROW15: track 0.00 -> 11.2 mm, vias 0 -> 1
- net ROW01: track 0.00 -> 10.7 mm, vias 0 -> 1
- net ROW13: track 0.00 -> 10.2 mm, vias 0 -> 1
- net ROW03: track 0.00 -> 9.65 mm, vias 0 -> 1
- net ROW14: track 0.00 -> 9.15 mm, vias 0 -> 1
- net ROW11: track 0.00 -> 9.15 mm, vias 0 -> 1
- net ROW05: track 0.00 -> 8.65 mm, vias 0 -> 1
- net ROW02: track 0.00 -> 8.65 mm, vias 0 -> 1
- net ROW12: track 0.00 -> 8.15 mm, vias 0 -> 1
- net ROW09: track 0.00 -> 8.15 mm, vias 0 -> 1
- net ROW07: track 0.00 -> 7.65 mm, vias 0 -> 1
- net ROW04: track 0.00 -> 7.65 mm, vias 0 -> 1
- net ROW10: track 0.00 -> 7.15 mm, vias 0 -> 1
- net ROW06: track 0.00 -> 6.65 mm, vias 0 -> 1
- net ROW08: track 0.00 -> 6.15 mm, vias 0 -> 1
Other:
- board size 197.6 x 230.1 mm -> 197.6 x 236.8 mm
- board text added: "forearm Back"
- board text added: "forearm Back: 2-layer flex. Electrodes on B.Cu under the B.Mask opening; FFC connector J1 on F.Cu. Eco1.User = PSA adhesive on the B.Cu side. Eco2.User = stiffener under the connector (on the B.Cu side of the tail)."
- board text removed: "forearm Back: 1-layer flex, copper on B.Cu. B.Mask = coverlay openings. Eco1.User = PSA adhesive (copper side). Eco2.User = tail stiffener (opposite side), total tail 0.30 +/-0.05 mm. 16-pin 0.5 mm FFC fingers."

Commit message: Iteration 2: forearm pad from the measured paper template, bicep rescaled
The forearm outline is now digitised from the paper template wrapped round
the wearer's forearm (FOREARM_TEMPLATE_MM, scaled by the ruler in the photo):
240 mm round the arm at the elbow end, 210 mm long, narrowing to the 50 mm
underside strap at the wrist, tails on the elbow-end edge. The bicep pad is
scaled to the same arm (180 mm long, 200 -> 175 mm wide); the chest halves
are unchanged. Boards carry "iter2" in their title block and summary.json,
and all Gerbers, footprints, previews and checks are regenerated.

Also adds the template photos and the updated documentation docx.

Co-Authored-By: Claude Fable 5.1 <noreply@anthropic.com>
Parts:
- moved J1 21.2 mm to (140.4, 15.5)
Connections:
- J1 pad 10: ROW09 -> ROW07
- J1 pad 11: ROW10 -> ROW08
- J1 pad 12: ROW11 -> ROW09
- J1 pad 13: ROW12 -> ROW10
- J1 pad 14: ROW13 -> ROW11
- J1 pad 15: ROW14 -> ROW12
- J1 pad 16: ROW15 -> ROW13
- J1 pad 2: ROW01 -> (no net)
- J1 pad 3: ROW02 -> ROW00
- J1 pad 4: ROW03 -> ROW01
- J1 pad 5: ROW04 -> ROW02
- J1 pad 6: ROW05 -> ROW03
- J1 pad 7: ROW06 -> ROW04
- J1 pad 8: ROW07 -> ROW05
- J1 pad 9: ROW08 -> ROW06
Routing:
- net ROW15: track 11.2 -> 0.00 mm, vias 1 -> 0
- net ROW14: track 9.15 -> 0.00 mm, vias 1 -> 0
- net ROW00: track 0.00 -> 8.65 mm, vias 0 -> 1
- net ROW05: track 8.65 -> 7.65 mm
- net ROW04: track 7.65 -> 6.65 mm
- net ROW03: track 9.65 -> 8.65 mm
- net ROW02: track 8.65 -> 7.65 mm
- net ROW01: track 10.7 -> 9.65 mm
- net ROW13: track 10.2 -> 11.1 mm
- net ROW12: track 8.15 -> 9.15 mm
- net ROW11: track 9.15 -> 10.1 mm
- net ROW10: track 7.15 -> 8.15 mm
- net ROW09: track 8.15 -> 9.15 mm
- net ROW08: track 6.15 -> 7.15 mm
- net ROW06: track 6.65 -> 6.15 mm
Other:
- board size 197.6 x 236.8 mm -> 240.9 x 230.7 mm
